Commit message: WIP #170 prototype TF refactoring

File: urdf/zed.urdf (robot description, URDF)
Before this commit: robot zed_camera, 4 links, 3 joints
Links:
- removed link zed_center
- removed link zed_depth_camera
- removed link zed_left_camera
- removed link zed_right_camera
- added link left_optical; visual cylinder length=.031 radius=0.007
- added link right_optical; visual cylinder length=.031 radius=0.007
- added link zed_camera; visual mesh filename=package://zed_wrapper/urdf/ZED.stl
Joints:
- removed joint zed_depth_camera_joint
- removed joint zed_left_camera_joint
- removed joint zed_right_camera_joint
- added joint left_optical_joint: type fixed, parent zed_camera, child left_optical, origin xyz=0 0.00 0 rpy=0 0 0
- added joint right_optical_joint: type fixed, parent zed_camera, child right_optical, origin xyz=0.12 0 0 rpy=0 0 0

File: urdf/zedm.urdf (robot description, URDF)
Before this commit: robot zedm_camera, 4 links, 3 joints
Links:
- removed link zed_center
- removed link zed_depth_camera
- removed link zed_left_camera
- removed link zed_right_camera
- added link left_optical
- added link right_optical
- added link zed_camera; visual mesh filename=package://zed_wrapper/urdf/ZEDM.stl
Joints:
- removed joint zed_depth_camera_joint
- removed joint zed_left_camera_joint
- removed joint zed_right_camera_joint
- added joint left_optical_joint: type fixed, parent zed_camera, child left_optical, origin xyz=0 0.00 0 rpy=0 0 0
- added joint right_optical_joint: type fixed, parent zed_camera, child right_optical, origin xyz=0.06 0 0 rpy=0 0 0
